File: PCB/dancbot pcb/_autosave-dancebot pcb design.kicad_pcb (KiCad board)
At the start: 2 copper layers, 27 parts, among them J1 ESP32-PICO-KIT-V4.1, J2 Voltage Regulator, J4 Pins, J6 Conn_01x04_Socket, J7 Conn_01x04_Socket, Q1 PMOS, Q2 PMOS, Q3 2N3904, Q5 PMOS, SW1 SP switch, SW2 SW_SPST

Commit message: Connections For Layout Revision 2
Other:
- board outline added: 62.5 x 55 mm
Changed lines of the file:
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@@
     )
   )
-  (gr_rect (start 182 56) (end 251 121)
-    (stroke (width 0.2) (type default)) (fill none) (layer "F.Cu"))
+  (gr_rect (start 182.5 57.5) (end 245 112.5)
+    (stroke (width 0.1) (type default)) (fill none) (layer "Edge.Cuts"))
   (segment (start 197.92 63) (end 192.92 68) (width 0.25) (layer "F.Cu") (net 3))
   (segment (start 223.885 60.635) (end 224.73 61.48) (width 0.25) (layer "F.Cu") (net 3))
