File: dancebot_pcb_rev4/PCB.kicad_pcb (KiCad board)
At the start: 2 copper layers, 63.5 x 53.3 mm, 30 parts, among them J1 Voltage Regulator, J10 NeoPixel Right Eye, J11 Rocker Switch, J2 IO14 servo 1, J3 IO13 servo 2, J4 IO12 servo 3, J5 IO15 servo 4, J6 IO18 servo 5 (hat), J8 Pins, J9 NeoPixel Left Eye, Q1 IRLML6402TRPBF, U1 IRLML2502TRPBF, U2 ESP32-DEVKITC-32U

Commit message: Current PCB Progress
Parts:
- removed TP5, TP6: TestPoint, TestPoint:TestPoint_Pad_2.0x2.0mm
- added C1: 4.7u, Capacitor_SMD:C_0805_2012Metric, F.Cu at (176.5, 64.0)
- added C2: 0.1u, Capacitor_SMD:C_0805_2012Metric, F.Cu at (180.5, 64.0)
- added C3: 0.1u, Capacitor_SMD:C_0805_2012Metric, F.Cu at (156.0, 108.5)
- added C4: 0.1u, Capacitor_SMD:C_0805_2012Metric, F.Cu at (182.0, 86.0)
- added C5: 10u, Capacitor_SMD:C_0805_2012Metric, F.Cu at (165.5, 112.5)
- added C6: 22u, Capacitor_SMD:C_0805_2012Metric, F.Cu at (165.5, 116.5)
- added C7: 22u, Capacitor_SMD:C_0805_2012Metric, F.Cu at (173.0, 110.5)
- added C8: 0.1u, Capacitor_SMD:C_0805_2012Metric, F.Cu at (176.0, 111.0)
- added C9: 1u, Capacitor_SMD:C_0805_2012Metric, F.Cu at (178.6, 122.0)
- added D1: LED, LED_SMD:LED_0805_2012Metric, F.Cu at (178.5, 107.0)
- added J7: UJ2-MIBH2-4-SMT-TR, UJ2-MIBH-4-SMT-TR:CUIDEVICES_UJ2-MIBH-4-SMT-TR, F.Cu at (192.5, 69.0)
- added Q2: S8050, Package_TO_SOT_THT:TO-92_Inline, F.Cu at (177.0, 79.0)
- added Q3: S8050, Package_TO_SOT_THT:TO-92_Inline, F.Cu at (191.6, 75.2)
- added R10: 10k, Resistor_SMD:R_0805_2012Metric, F.Cu at (184.4, 79.0)
- added R11: 2k, Resistor_SMD:R_0805_2012Metric, F.Cu at (176.9, 94.5)
- added R12: 2k, Resistor_SMD:R_0805_2012Metric, F.Cu at (181.5, 107.0)
- added R13: 10k, Resistor_SMD:R_0805_2012Metric, F.Cu at (173.0, 122.1)
- added R7: 22.1k, Resistor_SMD:R_0805_2012Metric, F.Cu at (172.1, 68.0)
- added R8: 47.5k, Resistor_SMD:R_0805_2012Metric, F.Cu at (167.6, 68.0)
- added R9: 10k, Resistor_SMD:R_0805_2012Metric, F.Cu at (184.4, 76.0)
- added SW1: RESET, Button_Switch_THT:KSA_Tactile_SPST, F.Cu at (171.5, 104.0)
- added SW2: BOOT, Button_Switch_THT:KSA_Tactile_SPST, F.Cu at (188.9, 86.1)
- added U3: ESP32-WROOM-32E__4MB_, ESP32-WROOM-32E__4MB_:XCVR_ESP32-WROOM-32E__4MB_, F.Cu at (159.8, 92.2)
- added U4: CP2102N-A02-GQFN28R, CP2102N-A02-GQFN28R:IC_CP2102N-A02-GQFN28R, F.Cu at (175.0, 73.0)
- Q1: footprint dancebot_parts:SOT95P237X112-3N -> IRLML6402TRPBF:SOT95P237X112-3N
- U1: footprint dancebot_parts:SOT23 -> IRLML2502TRPBF:SOT23
- U2: value ESP32-DEVKITC-32U -> AMS1117-3.3; footprint dancebot_parts:MODULE_ESP32-DEVKITC-32U -> AMS1117-3.3:SOT229P700X180-4N
- moved H1 108.4 mm to (150.5, 60.5), turned to 90 degrees
- moved J5 103.3 mm to (153.8, 76.6), turned to 180 degrees
- moved J4 89.8 mm to (158.5, 76.6), turned to 180 degrees
- moved J6 89.0 mm to (149.2, 76.6), turned to 180 degrees
- moved H4 88.7 mm to (194.5, 60.5), turned to 90 degrees
- moved J2 86.3 mm to (167.5, 76.6), turned to 180 degrees
- moved J3 81.4 mm to (163.0, 76.6), turned to 180 degrees
- moved TP1 78.8 mm to (160.0, 104.0), turned to -90 degrees
- moved U2 76.4 mm to (159.0, 115.0), turned to 90 degrees
- moved R3 64.9 mm to (172.0, 115.6), turned to 90 degrees
- moved H2 63.7 mm to (150.5, 115.0), turned to 90 degrees
- moved TP2 59.3 mm to (182.0, 98.4), turned to 180 degrees
- moved R2 54.3 mm to (175.0, 115.6), turned to -90 degrees
- moved R4 53.7 mm to (175.5, 99.5), turned to -90 degrees
- moved TP3 53.3 mm to (182.0, 94.4)
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Connections:
- D2 pad 1: Net-(D2-K) -> VBUS
- J2 pad 2: VOUT -> VBUS
- J3 pad 2: VOUT -> VBUS
- J4 pad 2: VOUT -> VBUS
- J5 pad 2: VOUT -> VBUS
- J6 pad 2: VOUT -> VBUS
- U2 pad 1: unconnected-(U2-3V3-Pad1) -> GND
- U2 pad 2: unconnected-(U2-EN-Pad2) -> 3v3
- U2 pad 3: unconnected-(U2-SENSOR_VP-Pad3) -> VBUS
- U2 pad 4: unconnected-(U2-SENSOR_VN-Pad4) -> (no net)
Routing:
- net BATT PWR: track 65.6 -> 0.00 mm, vias 1 -> 0
- net VOUT: track 62.6 -> 0.00 mm
- net NPRightEye: track 42.9 -> 0.00 mm
- net NPLeftEye: track 41.9 -> 0.00 mm
- net BATT ADC: track 38.2 -> 0.00 mm
- net BATT EN: track 30.6 -> 0.00 mm
- net Net-(J1-Pin_5): track 24.0 -> 0.00 mm
- net Net-(D2-K): track 14.8 -> 0.00 mm
- net D+: track 0.00 -> 11.8 mm, vias 0 -> 1
- net GND: track 10.9 -> 0.00 mm, vias 2 -> 0
- net D-: track 0.00 -> 8.27 mm
- net Net-(R4-Pad2): track 5.75 -> 0.00 mm
- net Net-(R1-Pad2): track 4.90 -> 0.00 mm
- net Net-(Q1-Pad3): track 4.10 -> 0.00 mm
- net Net-(Q1-Pad1): track 3.65 -> 0.00 mm
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- removed copper zone on B.Cu, net GND
Other:
- board size 63.5 x 53.3 mm -> 53.3 x 63.5 mm
- board text removed: "+5V"
- board text removed: "- +"
- board text removed: "Dancebot v3 Joy Chen Arsen Iman Toby Nguyen"
- board text removed: "GND"
- board text removed: "L R"
- board text removed: "Switch"
- board text removed: "VOUT GND BGND BPWR"
- board text removed: "^ GND PIN"
