File: dancebot_pcb_rev4/POWER.kicad_sch (KiCad schematic)
At the start: 32 parts, among them IC1 TPS63000IDRCRQ1, J1 BAT_IN, J2 PWR_SW

Commit message: search replaced mouser.co.uk with mouser.com
Parts:
- C1, C2: Mouser Price/Stock https://www.mouser.co.uk/ProductDetail/TAIYO-YUDEN/MCAST21G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 -> https://www.mouser.com/ProductDetail/TAIYO-YUDEN/MCAST21GSB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
- C3, C5, C8, C9: Mouser Price/Stock https://www.mouser.co.uk/ProductDetail/TDK/C1608X7T1A106M08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 -> https://www.mouser.com/ProductDetail/TDK/C1608X7T1A106M080A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
- C4, C6: Mouser Price/Stock https://www.mouser.co.uk/ProductDetail/KYOCERA-AVX/KAF21KR7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 -> https://www.mouser.com/ProductDetail/KYOCERA-AVX/KAF21KR72A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
- C7: Mouser Price/Stock https://www.mouser.co.uk/ProductDetail/TAIYO-YUDEN/JMK212BB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 -> https://www.mouser.com/ProductDetail/TAIYO-YUDEN/JMK212BBJ2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
- D1, D2: Mouser Price/Stock https://www.mouser.co.uk/ProductDetail/Texas-Instruments/LM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 -> https://www.mouser.com/ProductDetail/Texas-Instruments/LM66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
- D3: Mouser Price/Stock https://www.mouser.co.uk/ProductDetail/Panjit/SMF5.0A_R1_00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 -> https://www.mouser.com/ProductDetail/Panjit/SMF5.0A_R1_0000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
- IC1, PS1: Mouser Price/Stock https://www.mouser.co.uk/ProductDetail/Texas-Instruments/TP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 -> https://www.mouser.com/ProductDetail/Texas-Instruments/TPS6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
- L1, L2: Mouser Price/Stock https://www.mouser.co.uk/ProductDetail/TAIYO-YUDEN/NRS3015T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 -> https://www.mouser.com/ProductDetail/TAIYO-YUDEN/NRS3015T2R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
- R1: Mouser Price/Stock https://www.mouser.co.uk/ProductDetail/Vishay-Draloric/RCG0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 -> https://www.mouser.com/ProductDetail/Vishay-Draloric/RCG080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
- R2: Mouser Price/Stock https://www.mouser.co.uk/ProductDetail/Vishay-Dale/CRCW0805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 -> https://www.mouser.com/ProductDetail/Vishay-Dale/CRCW080510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
- R3: Mouser Price/Stock https://www.mouser.co.uk/ProductDetail/Bourns/CR0805-FX-100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 -> https://www.mouser.com/ProductDetail/Bourns/CR0805-FX-1004E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
- R4: Mouser Price/Stock https://www.mouser.co.uk/ProductDetail/KOA-Speer/SG73P2ATTD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 -> https://www.mouser.com/ProductDetail/KOA-Speer/SG73P2ATTD20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
Changed lines of the file:
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@@
 			)
 		)
-		(property "Mouser Price/Stock" "https://www.mouser.co.uk/ProductDetail/TAIYO-YUDEN/NRS3015T2R2MNGHV?qs=DpxmIIQLg%252BP8UFyXVw61Xw%3D%3D"
+		(property "Mouser Price/Stock" "https://www.mouser.com/ProductDetail/TAIYO-YUDEN/NRS3015T2R2MNGHV?qs=DpxmIIQLg%252BP8UFyXVw61Xw%3D%3D"
 			(at 748.59 31.75 0)
 			(effects
@@
 			)
 		)
-		(property "Mouser Price/Stock" "https://www.mouser.co.uk/ProductDetail/Bourns/CR0805-FX-1004ELF?qs=tknLyCMIRbOGJekSMom0SQ%3D%3D"
+		(property "Mouser Price/Stock" "https://www.mouser.com/ProductDetail/Bourns/CR0805-FX-1004ELF?qs=tknLyCMIRbOGJekSMom0SQ%3D%3D"
 			(at 198.12 719.38 0)
 			(effects
@@
 			)
 		)
-		(property "Mouser Price/Stock" "https://www.mouser.co.uk/ProductDetail/Vishay-Draloric/RCG0805100RJNEA?qs=vOeJqewp7jAa9buYzH8MLQ%3D%3D"
+		(property "Mouser Price/Stock" "https://www.mouser.com/ProductDetail/Vishay-Draloric/RCG0805100RJNEA?qs=vOeJqewp7jAa9buYzH8MLQ%3D%3D"
 			(at 148.59 713.03 0)
 			(effects
@@
 			)
 		)
-		(property "Mouser Price/Stock" "https://www.mouser.co.uk/ProductDetail/TDK/C1608X7T1A106M080AC?qs=Vi0JKjFBtYk5DbkZB9qYvg%3D%3D"
+		(property "Mouser Price/Stock" "https://www.mouser.com/ProductDetail/TDK/C1608X7T1A106M080AC?qs=Vi0JKjFBtYk5DbkZB9qYvg%3D%3D"
 			(at 104.14 648.26 0)
 			(effects
@@
 			)
 		)
-		(property "Mouser Price/Stock" "https://www.mouser.co.uk/ProductDetail/TAIYO-YUDEN/MCAST21GSB7105MTNB25?qs=tlsG%2FOw5FFgklVSELtG1Zg%3D%3D"
+		(property "Mouser Price/Stock" "https://www.mouser.com/ProductDetail/TAIYO-YUDEN/MCAST21GSB7105MTNB25?qs=tlsG%2FOw5FFgklVSELtG1Zg%3D%3D"
 			(at 55.88 704.14 0)
 			(effects
@@
 			)
 		)
-		(property "Mouser Price/Stock" "https://www.mouser.co.uk/ProductDetail/Vishay-Dale/CRCW0805100KFKEA?qs=LOX6nxTstibsf9am%252BHZOtQ%3D%3D"
+		(property "Mouser Price/Stock" "https://www.mouser.com/ProductDetail/Vishay-Dale/CRCW0805100KFKEA?qs=LOX6nxTstibsf9am%252BHZOtQ%3D%3D"
 			(at 748.59 26.67 0)
 			(effects
@@
 			)
 		)
-		(property "Mouser Price/Stock" "https://www.mouser.co.uk/ProductDetail/KYOCERA-AVX/KAF21KR72A104KL?qs=Jm2GQyTW%2FbiUCISqVwD%2FLA%3D%3D"
+		(property "Mouser Price/Stock" "https://www.mouser.com/ProductDetail/KYOCERA-AVX/KAF21KR72A104KL?qs=Jm2GQyTW%2FbiUCISqVwD%2FLA%3D%3D"
 			(at 110.49 746.05 0)
 			(effects
@@
 			)
 		)
-		(property "Mouser Price/Stock" "https://www.mouser.co.uk/ProductDetail/Texas-Instruments/LM66100DCKR?qs=vLWxofP3U2y2yPPrXoBBoA%3D%3D"
+		(property "Mouser Price/Stock" "https://www.mouser.com/ProductDetail/Texas-Instruments/LM66100DCKR?qs=vLWxofP3U2y2yPPrXoBBoA%3D%3D"
 			(at 77.47 699.06 0)
 			(effects
@@
 			)
 		)
-		(property "Mouser Price/Stock" "https://www.mouser.co.uk/ProductDetail/TAIYO-YUDEN/MCAST21GSB7105MTNB25?qs=tlsG%2FOw5FFgklVSELtG1Zg%3D%3D"
+		(property "Mouser Price/Stock" "https://www.mouser.com/ProductDetail/TAIYO-YUDEN/MCAST21GSB7105MTNB25?qs=tlsG%2FOw5FFgklVSELtG1Zg%3D%3D"
 			(at 55.88 743.51 0)
 			(effects
@@
 			)
 		)
-		(property "Mouser Price/Stock" "https://www.mouser.co.uk/ProductDetail/TDK/C1608X7T1A106M080AC?qs=Vi0JKjFBtYk5DbkZB9qYvg%3D%3D"
+		(property "Mouser Price/Stock" "https://www.mouser.com/ProductDetail/TDK/C1608X7T1A106M080AC?qs=Vi0JKjFBtYk5DbkZB9qYvg%3D%3D"
 			(at 203.2 719.38 0)
 			(effects
@@
 			)
 		)
-		(property "Mouser Price/Stock" "https://www.mouser.co.uk/ProductDetail/TAIYO-YUDEN/JMK212BBJ226MG8T?qs=hWgE7mdIu5QbK2Kg3NX%2FvQ%3D%3D"
+		(property "Mouser Price/Stock" "https://www.mouser.com/ProductDetail/TAIYO-YUDEN/JMK212BBJ226MG8T?qs=hWgE7mdIu5QbK2Kg3NX%2FvQ%3D%3D"
 			(at 171.45 650.8 0)
 			(effects
@@
 			)
 		)
-		(property "Mouser Price/Stock" "https://www.mouser.co.uk/ProductDetail/Panjit/SMF5.0A_R1_00001?qs=sPbYRqrBIVlx%2FHVv%252BUyL%252BQ%3D%3D"
+		(property "Mouser Price/Stock" "https://www.mouser.com/ProductDetail/Panjit/SMF5.0A_R1_00001?qs=sPbYRqrBIVlx%2FHVv%252BUyL%252BQ%3D%3D"
 			(at -523.8 41.91 0)
 			(effects
@@
 			)
 		)
-		(property "Mouser Price/Stock" "https://www.mouser.co.uk/ProductDetail/Texas-Instruments/LM66100DCKR?qs=vLWxofP3U2y2yPPrXoBBoA%3D%3D"
+		(property "Mouser Price/Stock" "https://www.mouser.com/ProductDetail/Texas-Instruments/LM66100DCKR?qs=vLWxofP3U2y2yPPrXoBBoA%3D%3D"
 			(at 77.47 738.43 0)
 			(effects
@@
 			)
 		)
-		(property "Mouser Price/Stock" "https://www.mouser.co.uk/ProductDetail/KOA-Speer/SG73P2ATTD2003F?qs=0U9fANxrh6nXGXRg%2FonPow%3D%3D"
+		(property "Mouser Price/Stock" "https://www.mouser.com/ProductDetail/KOA-Speer/SG73P2ATTD2003F?qs=0U9fANxrh6nXGXRg%2FonPow%3D%3D"
 			(at 198.12 729.54 0)
 			(effects
@@
 			)
 		)
-		(property "Mouser Price/Stock" "https://www.mouser.co.uk/ProductDetail/Texas-Instruments/TPS62163DSGR?qs=gXEV9p%2FxLgeWmbvztTvegw%3D%3D"
+		(property "Mouser Price/Stock" "https://www.mouser.com/ProductDetail/Texas-Instruments/TPS62163DSGR?qs=gXEV9p%2FxLgeWmbvztTvegw%3D%3D"
 			(at 137.16 640.64 0)
 			(effects
@@
 			)
 		)
-		(property "Mouser Price/Stock" "https://www.mouser.co.uk/ProductDetail/TAIYO-YUDEN/NRS3015T2R2MNGHV?qs=DpxmIIQLg%252BP8UFyXVw61Xw%3D%3D"
+		(property "Mouser Price/Stock" "https://www.mouser.com/ProductDetail/TAIYO-YUDEN/NRS3015T2R2MNGHV?qs=DpxmIIQLg%252BP8UFyXVw61Xw%3D%3D"
 			(at 757.48 81.28 0)
 			(effects
@@
 			)
 		)
-		(property "Mouser Price/Stock" "https://www.mouser.co.uk/ProductDetail/KYOCERA-AVX/KAF21KR72A104KL?qs=Jm2GQyTW%2FbiUCISqVwD%2FLA%3D%3D"
+		(property "Mouser Price/Stock" "https://www.mouser.com/ProductDetail/KYOCERA-AVX/KAF21KR72A104KL?qs=Jm2GQyTW%2FbiUCISqVwD%2FLA%3D%3D"
 			(at 143.51 724.46 0)
 			(effects
@@
 			)
 		)
-		(property "Mouser Price/Stock" "https://www.mouser.co.uk/ProductDetail/TDK/C1608X7T1A106M080AC?qs=Vi0JKjFBtYk5DbkZB9qYvg%3D%3D"
+		(property "Mouser Price/Stock" "https://www.mouser.com/ProductDetail/TDK/C1608X7T1A106M080AC?qs=Vi0JKjFBtYk5DbkZB9qYvg%3D%3D"
 			(at 210.82 719.38 0)
 			(effects
@@
 			)
 		)
-		(property "Mouser Price/Stock" "https://www.mouser.co.uk/ProductDetail/Texas-Instruments/TPS63000IDRCRQ1?qs=i6VRxKQL%2FYw6zzUuY%2FiBvw%3D%3D"
+		(property "Mouser Price/Stock" "https://www.mouser.com/ProductDetail/Texas-Instruments/TPS63000IDRCRQ1?qs=i6VRxKQL%2FYw6zzUuY%2FiBvw%3D%3D"
 			(at 175.26 701.6 0)
 			(effects
@@
 			)
 		)
-		(property "Mouser Price/Stock" "https://www.mouser.co.uk/ProductDetail/TDK/C1608X7T1A106M080AC?qs=Vi0JKjFBtYk5DbkZB9qYvg%3D%3D"
+		(property "Mouser Price/Stock" "https://www.mouser.com/ProductDetail/TDK/C1608X7T1A106M080AC?qs=Vi0JKjFBtYk5DbkZB9qYvg%3D%3D"
 			(at 130.81 716.84 0)
 			(effects
